File: PCB/K-Type.kicad_pcb (KiCad board)
At the start: 2 copper layers, 357.5 x 131.8 mm, 362 parts, among them J1 USBC, J2 USBC, P1 FLASH_HDR, P2 CONN_16, U1 MK20DX256VLH7, U2 TS3DS10224, U3 TS3USB30E, U4 IS31FL3733, U5 IS31FL3733, X1 CRYSTAL

Commit message: Removed bad traces; gotta redraw everything now
Routing:
- net /ledmatrix/LD1_SW8: track 372.4 -> 208.4 mm
- net /ledmatrix/LD1_SW11: track 376.9 -> 226.5 mm, vias 6 -> 5
- net /ledmatrix/LD1_SW7: track 388.4 -> 254.0 mm, vias 22 -> 14
- net /ledmatrix/LD1_SW5: track 379.0 -> 245.5 mm, vias 4 -> 2
- net /ledmatrix/LD2_SW2: track 380.8 -> 279.2 mm, vias 6 -> 4
- net /ledmatrix/LD1_SW1: track 447.9 -> 346.4 mm, vias 18 -> 11
- net /ledmatrix/LD2_SW7: track 615.6 -> 519.5 mm, vias 15 -> 12
- net /ledmatrix/LD1_SW10: track 390.5 -> 302.3 mm, vias 21 -> 14
- net /ledmatrix/LD2_SW3: track 379.6 -> 295.1 mm, vias 11 -> 10
- net /ledmatrix/LD2_SW1: track 390.1 -> 307.0 mm, vias 19 -> 15
- net /ledmatrix/LD1_SW2: track 430.7 -> 349.1 mm
- net /ledmatrix/LD2_SW9: track 603.8 -> 524.9 mm, vias 14 -> 12
- net /ledmatrix/LD1_SW4: track 386.9 -> 311.4 mm, vias 21 -> 18
- net /ledmatrix/LD2_SW5: track 376.6 -> 322.5 mm, vias 10 -> 9
- net /ledmatrix/LD1_CS15: track 135.7 -> 87.1 mm, vias 6 -> 2
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
Commit message: Making slow, painful progress
Routing:
- net /ledmatrix/LD2_SW10: track 246.4 -> 225.0 mm, vias 9 -> 11
- net /ledmatrix/LD2_SW11: track 261.2 -> 268.5 mm
- net /ledmatrix/LD2_CS4: track 427.1 -> 434.2 mm
- net /ledmatrix/LD2_SW12: track 223.4 -> 227.5 mm, vias 13 -> 15
- net /ledmatrix/LD1_SW2: track 349.1 -> 351.7 mm, vias 4 -> 6

Commit message: Making more, slow, painful progress
Routing:
- net /ledmatrix/LD2_SW9: track 524.9 -> 622.5 mm, vias 12 -> 14
- net /ledmatrix/LD2_SW7: track 519.5 -> 595.3 mm, vias 12 -> 16
- net /ledmatrix/LD2_SW12: track 227.5 -> 260.6 mm, vias 15 -> 18
- net /ledmatrix/LD2_SW10: track 225.0 -> 244.8 mm, vias 11 -> 14
- net /ledmatrix/LD1_CS16: track 377.2 -> 395.3 mm, vias 6 -> 8
- net /ledmatrix/LD1_SW3: track 407.1 -> 415.0 mm, vias 8 -> 12
- net /ledmatrix/LD2_CS8: track 424.1 -> 430.9 mm, vias 4 -> 6
- net /ledmatrix/LD2_SW8: track 694.6 -> 700.4 mm
- net /ledmatrix/LD2_SW11: track 268.5 -> 273.5 mm
- net /ledmatrix/LD2_CS13: track 435.2 -> 437.9 mm
- net /ledmatrix/LD2_CS12: track 308.1 -> 310.5 mm, vias 4 -> 6
- net /ledmatrix/LD1_SW2: track 351.7 -> 353.1 mm
- net /ledmatrix/LD2_CS3: track 402.2 -> 401.0 mm
- net /ledmatrix/LD2_CS2: track 392.5 -> 393.3 mm
- net /ledmatrix/LD2_CS16: track 316.3 -> 317.1 mm, vias 3 -> 5
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
Commit message: Saving before more work
Routing:
- net /ledmatrix/LD1_CS15: track 87.1 -> 119.0 mm, vias 2 -> 6
- net /ledmatrix/LD1_SW1: track 346.5 -> 371.5 mm, vias 11 -> 13
- net /ledmatrix/LD1_SW2: track 353.1 -> 376.8 mm, vias 6 -> 10
- net /ledmatrix/LD1_SW3: track 415.0 -> 425.7 mm, vias 12 -> 14
- net /ledmatrix/LD1_CS13: track 170.0 -> 173.8 mm, vias 6 -> 7
- net /ledmatrix/LD1_CS14: track 161.7 -> 165.4 mm, vias 6 -> 7
- net /ledmatrix/LD2_SW11: track 273.5 -> 276.5 mm
