File: PCB/K-Type.kicad_pcb (KiCad board)
At the start: 2 copper layers, 357.5 x 131.8 mm, 362 parts, among them J1 USBC, J2 USBC, P1 FLASH_HDR, P2 CONN_16, U1 MK20DX256VLH7, U2 TS3DS10224, U3 TS3USB30E, U4 IS31FL3733, U5 IS31FL3733, X1 CRYSTAL

Commit message: Halfway done?
Routing:
- net /ledmatrix/LD1_SW7: track 2.58 -> 406.2 mm, vias 0 -> 31
- net /ledmatrix/LD1_SW9: track 1.12 -> 360.4 mm
- net /ledmatrix/LD1_SW8: track 2.52 -> 312.3 mm
- net /ledmatrix/LD1_SW4: track 355.5 -> 429.8 mm, vias 28 -> 35
- net /ledmatrix/LD1_SW6: track 322.1 -> 391.4 mm, vias 0 -> 4
- net /ledmatrix/LD1_SW5: track 277.6 -> 340.6 mm, vias 0 -> 4
- net /ledmatrix/LD1_SW12: track 2.62 -> 26.6 mm
- net /ledmatrix/LD1_SW10: track 1.45 -> 24.2 mm, vias 0 -> 2
- net /ledmatrix/LD1_SW11: track 3.15 -> 23.6 mm
- net /mcu/INA-: track 288.8 -> 291.7 mm
- net /mcu/INA+: track 289.4 -> 292.3 mm
- net +5V: track 544.0 -> 544.8 mm
- net /Col10: track 403.7 -> 404.4 mm

Commit message: Saving progress
Routing:
- net /ledmatrix/LD2_SW6: track 1.82 -> 478.5 mm, vias 0 -> 26
- net /ledmatrix/LD2_SW4: track 1.50 -> 473.3 mm, vias 0 -> 26
- net /ledmatrix/LD2_SW5: track 1.30 -> 438.2 mm, vias 0 -> 30
- net /ledmatrix/LD2_SW1: track 1.27 -> 346.3 mm, vias 0 -> 24
- net /ledmatrix/LD1_SW10: track 24.2 -> 356.2 mm, vias 2 -> 29
- net /ledmatrix/LD2_SW3: track 1.05 -> 316.4 mm, vias 0 -> 2
- net /ledmatrix/LD1_SW12: track 26.6 -> 331.3 mm
- net /ledmatrix/LD2_SW2: track 1.68 -> 272.7 mm
- net /ledmatrix/LD1_SW11: track 23.6 -> 288.4 mm
- net /ledmatrix/LD2_SW9: track 252.4 -> 323.9 mm, vias 0 -> 4
- net /ledmatrix/LD2_SW7: track 255.5 -> 326.1 mm
- net /ledmatrix/LD2_SW8: track 245.8 -> 314.4 mm, vias 14 -> 18
- net /Row8: track 296.9 -> 294.5 mm
- net /Col9: track 490.5 -> 492.1 mm

Commit message: All RGB traces routed
Routing:
- net /ledmatrix/LD2_SW9: track 323.9 -> 547.4 mm, vias 4 -> 12
- net /ledmatrix/LD2_SW7: track 326.1 -> 546.1 mm, vias 14 -> 26
- net /ledmatrix/LD2_SW8: track 314.4 -> 526.9 mm, vias 18 -> 28
- net /ledmatrix/LD2_SW10: track 72.0 -> 219.7 mm, vias 4 -> 13
- net /ledmatrix/LD2_SW12: track 71.1 -> 217.8 mm, vias 0 -> 4
- net /ledmatrix/LD2_SW11: track 68.3 -> 213.1 mm, vias 4 -> 13
- net /ledmatrix/LD2_SW2: track 272.7 -> 407.1 mm, vias 0 -> 6
- net /ledmatrix/LD2_SW3: track 316.4 -> 422.9 mm, vias 2 -> 6
- net /ledmatrix/LD2_SW1: track 346.3 -> 446.0 mm, vias 24 -> 27
- net /ledmatrix/LD1_SW3: track 338.6 -> 410.8 mm, vias 0 -> 2
- net /ledmatrix/LD1_SW2: track 295.5 -> 367.0 mm, vias 0 -> 4
- net /ledmatrix/LD1_SW1: track 367.9 -> 435.3 mm, vias 26 -> 29
- net /ledmatrix/LD1_SW7: track 406.2 -> 462.4 mm, vias 31 -> 36
- net /ledmatrix/LD1_SW8: track 312.3 -> 366.8 mm, vias 0 -> 2
- net /ledmatrix/LD1_SW9: track 360.4 -> 414.1 mm, vias 0 -> 2
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
Commit message: Finished routing interboard connections
Routing:
- net /ledmatrix/LD1_CS3: track 2.68 -> 269.7 mm, vias 0 -> 4
- net /ledmatrix/LD1_CS4: track 1.20 -> 253.5 mm, vias 0 -> 4
- net /ledmatrix/LD2_CS16: track 1.81 -> 235.2 mm, vias 0 -> 12
- net /ledmatrix/LD1_CS5: track 3.92 -> 236.2 mm, vias 0 -> 8
- net /ledmatrix/LD1_CS6: track 2.11 -> 218.4 mm, vias 0 -> 8
- net /ledmatrix/LD2_CS15: track 1.77 -> 202.8 mm, vias 0 -> 12
- net /ledmatrix/LD1_CS7: track 2.34 -> 200.9 mm, vias 0 -> 6
- net /ledmatrix/LD1_CS8: track 1.87 -> 181.4 mm, vias 0 -> 6
- net /ledmatrix/LD2_CS5: track 1.36 -> 175.4 mm, vias 0 -> 6
- net /ledmatrix/LD1_CS9: track 3.48 -> 161.8 mm, vias 0 -> 6
- net /ledmatrix/LD2_CS14: track 0.96 -> 158.3 mm, vias 0 -> 10
- net /ledmatrix/LD2_CS6: track 0.93 -> 154.4 mm, vias 0 -> 6
- net /ledmatrix/LD1_CS10: track 2.58 -> 146.8 mm, vias 0 -> 6
- net /ledmatrix/LD2_CS7: track 3.69 -> 132.7 mm, vias 0 -> 6
- net /ledmatrix/LD2_CS13: track 1.52 -> 125.0 mm, vias 0 -> 10
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
Commit message: All traces except for cross traces routed
Routing:
- net /ledmatrix/LD2_SW9: track 547.4 -> 805.7 mm, vias 12 -> 20
- net /ledmatrix/LD2_SW8: track 526.9 -> 775.2 mm, vias 28 -> 36
- net /ledmatrix/LD2_SW7: track 546.1 -> 791.7 mm, vias 26 -> 34
- net /ledmatrix/LD2_SW11: track 213.1 -> 353.3 mm, vias 13 -> 17
- net /ledmatrix/LD2_SW10: track 219.7 -> 358.3 mm, vias 13 -> 19
- net /ledmatrix/LD2_SW12: track 217.8 -> 345.6 mm, vias 4 -> 8
- net /ledmatrix/LD1_SW10: track 377.0 -> 491.5 mm, vias 29 -> 42
- net /ledmatrix/LD1_SW12: track 359.4 -> 470.5 mm, vias 2 -> 10
- net /ledmatrix/LD1_SW2: track 367.0 -> 468.6 mm, vias 4 -> 20
- net /ledmatrix/LD1_SW3: track 410.8 -> 509.9 mm, vias 2 -> 18
- net /ledmatrix/LD1_SW1: track 435.3 -> 529.7 mm, vias 29 -> 44
- net /ledmatrix/LD1_SW11: track 314.1 -> 407.7 mm, vias 2 -> 14
- net /ledmatrix/LD2_SW1: track 446.0 -> 528.4 mm, vias 27 -> 37
- net /ledmatrix/LD2_SW2: track 407.1 -> 489.2 mm, vias 6 -> 17
- net /ledmatrix/LD2_SW3: track 422.9 -> 498.8 mm, vias 6 -> 12
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