File: PCB/K-Type_original.kicad_pcb (KiCad board)
At the start: 2 copper layers, 357.5 x 131.8 mm, 362 parts, among them J1 USBC, J2 USBC, P1 FLASH_HDR, P2 CONN_16, U1 MK20DX256VLH7, U2 TS3DS10224, U3 TS3USB30E, U4 IS31FL3733, U5 IS31FL3733, X1 CRYSTAL

Commit message: Adding newer attempt at PCB
Routing:
- net /ledmatrix/LD2_SW8: track 245.8 -> 707.0 mm, vias 14 -> 16
- net /ledmatrix/LD2_CS14: track 0.96 -> 461.5 mm, vias 0 -> 5
- net /ledmatrix/LD2_CS5: track 1.36 -> 438.8 mm, vias 0 -> 6
- net /ledmatrix/LD2_CS13: track 1.52 -> 437.4 mm, vias 0 -> 6
- net /ledmatrix/LD2_CS7: track 3.69 -> 436.7 mm, vias 0 -> 4
- net /ledmatrix/LD2_CS4: track 1.38 -> 430.5 mm, vias 0 -> 6
- net /ledmatrix/LD2_CS8: track 3.28 -> 431.1 mm, vias 0 -> 4
- net /ledmatrix/LD2_CS15: track 1.77 -> 425.0 mm, vias 0 -> 5
- net /ledmatrix/LD2_CS6: track 0.93 -> 409.2 mm, vias 0 -> 6
- net /ledmatrix/LD1_CS2: track 1.43 -> 406.2 mm, vias 0 -> 5
- net /ledmatrix/LD2_CS3: track 2.86 -> 405.0 mm, vias 0 -> 6
- net /ledmatrix/LD1_CS1: track 2.26 -> 401.8 mm, vias 0 -> 8
- net /ledmatrix/LD2_CS2: track 2.21 -> 395.6 mm, vias 0 -> 6
- net /ledmatrix/LD2_CS1: track 1.76 -> 394.5 mm, vias 0 -> 8
- net /ledmatrix/LD1_SW10: track 1.45 -> 390.5 mm, vias 0 -> 21
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Other:
- net class Default: trace_width 0.216 -> 0.25
